File: hardware/kicad/Neopixel USB.kicad_pcb (KiCad board)
At the start: 2 copper layers, 31.6 x 12.5 mm, 13 parts, among them U1 ATtiny85-20S

Commit message: Mise à jour du schema
Parts:
- removed D2: 3V6, Diode_SMD:D_SOD-123
- removed D3: WS2812B, LED_SMD:LED_WS2812B_PLCC4_5.0x5.0mm_P3.2mm
- removed REF**: Tortue, arthur:Tortue
- added C2: 100nF, Capacitor_SMD:C_0603_1608Metric, F.Cu at (32.6, 35.1)
- added C4: 100nF, Capacitor_SMD:C_0603_1608Metric, B.Cu at (32.1, 34.8)
- added C5: 100nF, Capacitor_SMD:C_0603_1608Metric, B.Cu at (32.1, 43.5)
- added C6: 100nF, Capacitor_SMD:C_0603_1608Metric, B.Cu at (43.6, 40.9)
- added C7: 100nF, Capacitor_SMD:C_0603_1608Metric, B.Cu at (43.6, 37.3)
- added C8: 100nF, Capacitor_SMD:C_0603_1608Metric, B.Cu at (42.9, 34.7)
- added J1: USB C Male 24 pins U261-241N-4BS60, arthur:USB-C male 24 pins XKB_U261-241N-4BS60, F.Cu at (27.4, 39.1)
- added TP1: BOOT0, arthur:TestPoint_Pad_D1.0mm_1, F.Cu at (36.9, 37.8)
- added TP2: SWDIO, arthur:TestPoint_Pad_D1.0mm_1, F.Cu at (35.6, 37.8)
- added TP3: SWCLK, arthur:TestPoint_Pad_D1.0mm_1, F.Cu at (35.6, 39.1)
- added TP4: NRST, arthur:TestPoint_Pad_D1.0mm_1, F.Cu at (35.6, 40.4)
- added TP5: 3.3V, arthur:TestPoint_Pad_D1.0mm_1, F.Cu at (36.9, 39.1)
- added TP6: GND, arthur:TestPoint_Pad_D1.0mm_1, F.Cu at (36.9, 40.4)
- C1, C3: footprint Capacitor_SMD:C_0603_1608Metric_Pad1.08x0.95mm_HandSolder -> Capacitor_SMD:C_0603_1608Metric
- D1: value 3V6 -> WS2812B; footprint Diode_SMD:D_SOD-123 -> LED_SMD:LED_WS2812B_PLCC4_5.0x5.0mm_P3.2mm
- R1: value 10k -> 1.5k; footprint Resistor_SMD:R_0603_1608Metric_Pad0.98x0.95mm_HandSolder -> Resistor_SMD:R_0603_1608Metric
- R2: value 68 -> 5.1K; footprint Resistor_SMD:R_0603_1608Metric_Pad0.98x0.95mm_HandSolder -> Resistor_SMD:R_0603_1608Metric
- R3: value 68 -> 5.1K; footprint Resistor_SMD:R_0603_1608Metric_Pad0.98x0.95mm_HandSolder -> Resistor_SMD:R_0603_1608Metric; moved to B.Cu
- R4: value 1.5k -> 470; footprint Resistor_SMD:R_0603_1608Metric_Pad0.98x0.95mm_HandSolder -> Resistor_SMD:R_0603_1608Metric
- R5: value 470 -> 10k; footprint Resistor_SMD:R_0603_1608Metric_Pad0.98x0.95mm_HandSolder -> Resistor_SMD:R_0603_1608Metric
- U1: value ATtiny85-20S -> MCP1700x-330xxTT; footprint Package_SO:SOIC-8_5.3x5.3mm_P1.27mm -> Package_TO_SOT_SMD:SOT-23
- U2: value ~ -> STM32F072CBTx; footprint arthur:USB A Male PCB -> Package_QFP:LQFP-48_7x7mm_P0.5mm; moved to B.Cu
- moved C1 29.7 mm to (32.6, 40.1)
- moved R5 27.7 mm to (36.3, 35.1)
- moved R2 26.5 mm to (32.6, 43.1)
- moved U1 24.7 mm to (32.6, 37.5), turned to 180 degrees
- moved R3 23.8 mm to (31.1, 37.2), turned to -90 degrees
- moved R1 20.4 mm to (32.6, 41.6), turned to 0 degrees
- moved R4 19.5 mm to (41.3, 43.5)
- moved C3 18.3 mm to (41.3, 34.7), turned to 180 degrees
- moved U2 18.1 mm to (37.5, 39.1), turned to 180 degrees
- moved D1 17.2 mm to (41.3, 39.1), turned to -90 degrees
Connections:
- C1 pad 1: VCC -> +5V
- C3 pad 1: VCC -> +5V
- D1 pad 1: Net-(D1-K) -> +5V
- D1 pad 2: GND -> unconnected-(D1-DOUT-Pad2)
- R1 pad 1: Net-(U1-~{RESET}/PB5) -> USB_P
- R1 pad 2: VCC -> +3.3V
- R2 pad 1: PB3 -> GND
- R2 pad 2: Net-(D1-K) -> Net-(J1-CC)
- R3 pad 1: PB4 -> GND
- R3 pad 2: Net-(D2-K) -> Net-(J1-VCONN)
- R4 pad 1: VCC -> LED
- R4 pad 2: Net-(D1-K) -> Net-(D1-DIN)
- R5 pad 1: PB2 -> GND
- R5 pad 2: Net-(D3-DIN) -> BOOT0
- U1 pad 1: Net-(U1-~{RESET}/PB5) -> GND
- U1 pad 2: PB3 -> +3.3V
- U1 pad 3: PB4 -> +5V
- U2 pad 1: VCC -> +3.3V
- U2 pad 2: Net-(D1-K) -> unconnected-(U2-PC13-Pad2)
- U2 pad 3: Net-(D2-K) -> unconnected-(U2-PC14-Pad3)
- U2 pad 4: GND -> unconnected-(U2-PC15-Pad4)
Routing:
- net VCC: track 41.8 -> 0.00 mm, vias 3 -> 0
- net +3.3V: track 0.00 -> 39.7 mm, vias 0 -> 3
- net +5V: track 0.00 -> 32.4 mm, vias 0 -> 5
- net Net-(D1-K): track 17.7 -> 0.00 mm
- net Net-(D2-K): track 13.6 -> 0.00 mm
- net USB_P: track 0.00 -> 10.7 mm, vias 0 -> 1
- net LED: track 0.00 -> 10.2 mm, vias 0 -> 1
- net PB4: track 10.1 -> 0.00 mm
- net PB3: track 9.98 -> 0.00 mm
- net PB2: track 8.02 -> 0.00 mm
- net USB_N: track 0.00 -> 7.90 mm, vias 0 -> 1
- net NRST: track 0.00 -> 6.49 mm, vias 0 -> 1
- net SWCLK: track 0.00 -> 5.07 mm, vias 0 -> 1
- net BOOT0: track 0.00 -> 4.93 mm, vias 0 -> 2
- net Net-(J1-CC): track 0.00 -> 4.79 mm
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Other:
- board size 31.6 x 12.5 mm -> 16 x 10.7 mm
